File: hardware/ESP8266_Single_RGB_RevA.brd (EAGLE design)
At the start: 72.1 x 55.2 mm, 41 parts, among them IC1 ESP-12E/F, J1 POWER_JACKPTH_LOCK, J2 B G R +, J4 G S V, Q1 IRF520, Q2 IRF520, Q3 IRF520, T1 2N3904, T2 2N3904, T3 2N3904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

Commit message: fix R16 - NOT NEEDED at ALL
Parts:
- R19: value 10k -> NOT NEEDED !!!
Changed lines of the file:
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@@
 <attribute name="VALUE" x="62.5094" y="24.765" size="1.27" layer="27" ratio="10"/>
 </element>
-<element name="R19" library="rcl" library_urn="urn:adsk.eagle:library:334" package="0207/10" package3d_urn="urn:adsk.eagle:package:23491/2" value="10k" x="38.1" y="30.48" smashed="yes" rot="R180">
+<element name="R19" library="rcl" library_urn="urn:adsk.eagle:library:334" package="0207/10" package3d_urn="urn:adsk.eagle:package:23491/2" value="NOT NEEDED !!!" x="38.1" y="30.48" smashed="yes" rot="R180">
 <attribute name="NAME" x="41.148" y="28.956" size="1.27" layer="25" ratio="10" rot="R180"/>
 <attribute name="POPULARITY" value="81" x="-31.75" y="118.11" size="1.778" layer="27" rot="R180" display="off"/>
