File: hardware/ESP8266_Single_RGB_RevB.brd (EAGLE design)
At the start: 72.1 x 55.2 mm, 47 parts, among them IC1 ESP-12E/F, IC2 LM2575-3.3S, J1 POWER_JACKPTH_LOCK, J2 B G R +, J4 G S V, Q1 IRF520, Q2 IRF520, Q3 IRF520, T1 2N3904, T2 2N3904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

Commit message: RevB more
Parts:
- R2, R3, R5, R6, R8, R9: value 1k -> 10k
Changed lines of the file:
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@@
 <attribute name="VALUE" x="40.3606" y="31.115" size="1.27" layer="27" ratio="10" rot="R180"/>
 </element>
-<element name="R2" library="rcl" library_urn="urn:adsk.eagle:library:334" package="0207/10" package3d_urn="urn:adsk.eagle:package:23491/2" value="1k" x="63.5" y="17.78" smashed="yes" rot="R90">
+<element name="R2" library="rcl" library_urn="urn:adsk.eagle:library:334" package="0207/10" package3d_urn="urn:adsk.eagle:package:23491/2" value="10k" x="63.5" y="17.78" smashed="yes" rot="R90">
 <attribute name="NAME" x="61.976" y="14.732" size="1.27" layer="25" ratio="10" rot="R90"/>
 <attribute name="POPULARITY" value="81" x="133.35" y="91.44" size="1.778" layer="27" rot="R90" display="off"/>
@@
 <attribute name="VALUE" x="56.8706" y="46.355" size="1.27" layer="27" ratio="10" rot="R180"/>
 </element>
-<element name="R3" library="rcl" library_urn="urn:adsk.eagle:library:334" package="0207/10" package3d_urn="urn:adsk.eagle:package:23491/2" value="1k" x="59.69" y="17.78" smashed="yes" rot="R90">
+<element name="R3" library="rcl" library_urn="urn:adsk.eagle:library:334" package="0207/10" package3d_urn="urn:adsk.eagle:package:23491/2" value="10k" x="59.69" y="17.78" smashed="yes" rot="R90">
 <attribute name="NAME" x="58.166" y="14.732" size="1.27" layer="25" ratio="10" rot="R90"/>
 <attribute name="POPULARITY" value="81" x="137.16" y="36.83" size="1.778" layer="27" rot="R90" display="off"/>
@@
 <attribute name="VALUE" x="42.1894" y="24.765" size="1.27" layer="27" ratio="10"/>
 </element>
-<element name="R5" library="rcl" library_urn="urn:adsk.eagle:library:334" package="0207/10" package3d_urn="urn:adsk.eagle:package:23491/2" value="1k" x="43.18" y="17.78" smashed="yes" rot="R90">
+<element name="R5" library="rcl" library_urn="urn:adsk.eagle:library:334" package="0207/10" package3d_urn="urn:adsk.eagle:package:23491/2" value="10k" x="43.18" y="17.78" smashed="yes" rot="R90">
 <attribute name="NAME" x="41.656" y="14.732" size="1.27" layer="25" ratio="10" rot="R90"/>
 <attribute name="POPULARITY" value="81" x="120.65" y="62.23" size="1.778" layer="27" rot="R90" display="off"/>
@@
 <attribute name="VALUE" x="43.815" y="15.5194" size="1.27" layer="27" ratio="10" rot="R90"/>
 </element>
-<element name="R6" library="rcl" library_urn="urn:adsk.eagle:library:334" package="0207/10" package3d_urn="urn:adsk.eagle:package:23491/2" value="1k" x="39.37" y="17.78" smashed="yes" rot="R90">
+<element name="R6" library="rcl" library_urn="urn:adsk.eagle:library:334" package="0207/10" package3d_urn="urn:adsk.eagle:package:23491/2" value="10k" x="39.37" y="17.78" smashed="yes" rot="R90">
 <attribute name="NAME" x="37.846" y="14.732" size="1.27" layer="25" ratio="10" rot="R90"/>
 <attribute name="POPULARITY" value="81" x="116.84" y="74.93" size="1.778" layer="27" rot="R90" display="off"/>
@@
 <attribute name="VALUE" x="21.8694" y="24.765" size="1.27" layer="27" ratio="10"/>
 </element>
-<element name="R8" library="rcl" library_urn="urn:adsk.eagle:library:334" package="0207/10" package3d_urn="urn:adsk.eagle:package:23491/2" value="1k" x="22.86" y="17.78" smashed="yes" rot="R90">
+<element name="R8" library="rcl" library_urn="urn:adsk.eagle:library:334" package="0207/10" package3d_urn="urn:adsk.eagle:package:23491/2" value="10k" x="22.86" y="17.78" smashed="yes" rot="R90">
 <attribute name="NAME" x="21.336" y="14.732" size="1.27" layer="25" ratio="10" rot="R90"/>
 <attribute name="POPULARITY" value="81" x="100.33" y="100.33" size="1.778" layer="27" rot="R90" display="off"/>
@@
 <attribute name="VALUE" x="23.495" y="15.5194" size="1.27" layer="27" ratio="10" rot="R90"/>
 </element>
-<element name="R9" library="rcl" library_urn="urn:adsk.eagle:library:334" package="0207/10" package3d_urn="urn:adsk.eagle:package:23491/2" value="1k" x="19.05" y="17.78" smashed="yes" rot="R90">
+<element name="R9" library="rcl" library_urn="urn:adsk.eagle:library:334" package="0207/10" package3d_urn="urn:adsk.eagle:package:23491/2" value="10k" x="19.05" y="17.78" smashed="yes" rot="R90">
 <attribute name="NAME" x="17.526" y="14.732" size="1.27" layer="25" ratio="10" rot="R90"/>
 <attribute name="POPULARITY" value="81" x="101.6" y="36.83" size="1.778" layer="27" rot="R90" display="off"/>
