File: hardware/ESP8266_Single_RGB_RevB.brd (EAGLE design)
At the start: 72.1 x 55.2 mm, 47 parts, among them IC1 ESP-12E/F, IC3 LM2594, J1 POWER_JACKPTH_LOCK, J2 B G R +, J4 G S V, Q1 IRF520, Q2 IRF520, Q3 IRF520, T1 2N3904, T2 2N3904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

Commit message: ESP8266 Single RevB fixed, Gerbers added
Parts:
- L1: value 100uH -> DR74-100uH; device SparkFun-Coils:INDUCTOR_4X4MM -> inductors:DR74
- moved R4 3.81 mm to (40.6, 25.4)
- moved L1 1.62 mm to (50.8, 27.3), turned to 180 degrees
Connections:
- net +3V3: now also L1.2; no longer L1.P$2
- net N$15: now also L1.1; no longer L1.P$1
Routing:
- net BOOT/SW1: track 17.6 -> 51.0 mm
- net CH1_OUT: track 11.9 -> 42.9 mm, vias 0 -> 3
- net CH3_OUT: track 2.54 -> 30.1 mm, vias 0 -> 1
- net +3V3: track 89.0 -> 115.7 mm, vias 0 -> 1
- net RESET: track 3.96 -> 30.5 mm, vias 0 -> 1
- net CH2_OUT: track 8.98 -> 29.7 mm, vias 0 -> 2
- net N$11: track 6.35 -> 7.93 mm
- net N$15: track 9.19 -> 10.5 mm
- net +VIN: track 112.9 -> 111.6 mm
