File: hardware/ESP8266_Single_RGB_RevC.sch (EAGLE design)
At the start: 47 parts, among them IC1 ESP-12E/F, IC3 LM2594, J1 POWER_JACKPTH_LOCK, J2 B G R +, J4 G S V, Q1 IRF520, Q2 IRF520, Q3 IRF520, T1 2N3904, T2 2N3904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

Commit message: RevC Ok
Parts:
- added C7: 4.7n, rcl:C-EUC0805
- added R10: 1.5k, rcl:R-EU_M0805
- added R11: 910, rcl:R-EU_R0805
Connections:
- new net N$5: C7.1, IC3.FB, R10.2, R11.1
- net +3V3: now also C7.2, R10.1; no longer IC3.FB
- net GND: now also R11.2
